Commit message: removed base_footprint

File: nuturtle_description/urdf/diff_drive.urdf.xacro (robot description, xacro)
@@ -9,5 +9,5 @@
 <xacro:property name="caster_radius" value="${(wheel_radius - chassis_thickness/2)/2}" />
 <!-- BASE-FOOTPRINT -->
-<link name="base_footprint"/>
+<!-- <link name="base_footprint"/> -->
 <!-- chassis -->
 <link name="base_link" >
@@ -57,9 +57,9 @@
 </link>
 <!-- joints -->
-<joint name="base" type="fixed">
+<!-- <joint name="base" type="fixed">
   <origin xyz="0 0 ${wheel_radius}" rpy="0 0 0" />
   <parent link="base_footprint"/>
   <child link="base_link" />
-</joint>
+</joint> -->
 <joint name="left_wheel_axle" type="continuous">
   <origin xyz="0 ${wheel_base/2} 0" rpy="0 0 0" />

Commit message: type

File: nuturtle_description/urdf/diff_drive.urdf.xacro (robot description, xacro)
@@ -7,9 +7,21 @@
 <xacro:property name="wheel_radius" value="${props['wheel_radius']}" />
 <xacro:property name="wheel_width" value="${props['wheel_width']}" />
-<xacro:property name="caster_radius" value="${(wheel_radius - chassis_thickness/2)/2}" />
+<xacro:property name="wheel_axle_offset" value="${props['wheel_axle_offset']}"/>
+<xacro:property name="caster_radius" value="${(wheel_radius - wheel_axle_offset)/2}" />
+<!-- mass of chassis -->
+<xacro:property name="M" value="${0.04}" />
+<!-- mass of wheel  -->
+<xacro:property name="m" value="${0.03}" />
 <!-- BASE-FOOTPRINT -->
-<!-- <link name="base_footprint"/> -->
+<link name="base_footprint"/>
+<!-- Base Scan -->
+<link name="base_scan"/>
 <!-- chassis -->
 <link name="base_link" >
+  <inertial>
+    <origin xyz="${chassis_length/2 - wheel_radius} 0 0" rpy="0 0 0"/>
+    <mass value="${0.04}"/>
+    <inertia ixx="${1/12*M*(chassis_length**2+chassis_thickness**2)}"  ixy="0"  ixz="0" iyy="${1/12*M*((wheel_base - wheel_width)**2+chassis_thickness**2)}" iyz="0" izz="${1/12*M*(chassis_length**2+(wheel_base - wheel_width)**2)}" />
+  </inertial>
   <visual>
     <origin xyz="${chassis_length/2 - wheel_radius} 0 0" rpy="0 0 0" />
@@ -21,7 +33,18 @@
     </material>
   </visual>
+  <collision>
+    <origin xyz="${chassis_length/2 - wheel_radius} 0 0" rpy="0 0 0"/>
+    <geometry>
+      <box size="${chassis_length} ${wheel_base - wheel_width} ${chassis_thickness}" />
+    </geometry>
+  </collision>
 </link>
 <!-- left wheel -->
 <link name="left_wheel">
+  <inertial>
+    <origin xyz="0 0 0" rpy="${-pi/2} 0 0"/>
+    <mass value="${m}"/>
+    <inertia ixx="${1/12*m*(3*wheel_radius**2 + wheel_width**2)}"  ixy="0"  ixz="0" iyy="${1/12*m*(3*wheel_radius**2 + wheel_width**2)}" iyz="0" izz="${0.5*m*wheel_radius**2}" />
+  </inertial>
   <visual>
     <origin xyz="0 0 0" rpy="${-pi/2} 0 0" />
@@ -33,7 +56,18 @@
     </material>
   </visual>
+  <collision>
+    <origin xyz="0 0 0" rpy="${-pi/2} 0 0"/>
+    <geometry>
+      <cylinder radius="${wheel_radius}" length="${wheel_width}" />
+    </geometry>
+  </collision>
 </link>
 <!-- right wheel -->
 <link name="right_wheel">
+  <inertial>
+    <origin xyz="0 0 0" rpy="${pi/2} 0 0"/>
+    <mass value="${m}"/>
+    <inertia ixx="${1/12*m*(3*wheel_radius**2 + wheel_width**2)}"  ixy="0"  ixz="0" iyy="${1/12*m*(3*wheel_radius**2 + wheel_width**2)}" iyz="0" izz="${0.5*m*wheel_radius**2}" />
+  </inertial>
   <visual>
     <origin xyz="0 0 0" rpy="${pi/2} 0 0" />
@@ -45,4 +79,10 @@
     </material>
   </visual>
+  <collision>
+    <origin xyz="0 0 0" rpy="${pi/2} 0 0"/>
+    <geometry>
+      <cylinder radius="${wheel_radius}" length="${wheel_width}" />
+    </geometry>
+  </collision>
 </link>
 <!-- caster wheel -->
@@ -55,13 +95,26 @@
     <material name="Black" />
   </visual>
+  <collision>
+    <origin xyz="0 0 0" rpy="0 0 0"/>
+    <geometry>
+      <sphere radius="${caster_radius}" />
+    </geometry>
+  </collision>
 </link>
 <!-- joints -->
-<!-- <joint name="base" type="fixed">
-  <origin xyz="0 0 ${wheel_radius}" rpy="0 0 0" />
+<joint name="base" type="fixed">
+  <!-- <origin xyz="${-chassis_length/2 + chassis_length/2 - wheel_radius} 0 ${chassis_thickness/2 - wheel_axle_offset + wheel_radius}" rpy="0 0 0" /> -->
+  <origin xyz="${-wheel_radius} 0 ${chassis_thickness/2 - wheel_axle_offset + wheel_radius}" rpy="0 0 0" />
   <parent link="base_footprint"/>
   <child link="base_link" />
-</joint> -->
+</joint>
+<joint name="base_lidar" type="fixed">
+  <origin xyz="0 0 ${chassis_thickness/2}" rpy="0 0 0" />
+  <axis xyz="0 1 0"/>
+  <parent link="base_link" />
+  <child link="base_scan" />
+</joint>
 <joint name="left_wheel_axle" type="continuous">
-  <origin xyz="0 ${wheel_base/2} 0" rpy="0 0 0" />
+  <origin xyz="0 ${wheel_base/2} ${-chassis_thickness/2 + wheel_axle_offset}" rpy="0 0 0" />
   <axis xyz="0 1 0"/>
   <parent link="base_link" />
@@ -69,5 +122,5 @@
 </joint>
 <joint name="right_wheel_axle" type="continuous">
-  <origin xyz="0 ${-wheel_base/2} 0" rpy="0 0 0" />
+  <origin xyz="0 ${-wheel_base/2} ${-chassis_thickness/2 + wheel_axle_offset}" rpy="0 0 0" />
   <axis xyz="0 1 0"/>
   <parent link="base_link" />
@@ -75,5 +128,5 @@
 </joint>
 <joint name="caster_joint" type="fixed">
-  <origin xyz="${chassis_length-wheel_radius-caster_radius} 0 ${-chassis_thickness/2-caster_radius}" rpy="0 0 0" />
+  <origin xyz="${chassis_length - wheel_radius - caster_radius} 0 ${-chassis_thickness/2 - caster_radius}" rpy="0 0 0" />
   <parent link="base_link" />
   <child link="caster" />

Commit message: updated mass

File: nuturtle_description/urdf/diff_drive.urdf.xacro (robot description, xacro)
@@ -10,16 +10,16 @@
 <xacro:property name="caster_radius" value="${(wheel_radius - wheel_axle_offset)/2}" />
 <!-- mass of chassis -->
-<xacro:property name="M" value="${0.04}" />
+<xacro:property name="M" value="${0.94}" />
 <!-- mass of wheel  -->
 <xacro:property name="m" value="${0.03}" />
 <!-- BASE-FOOTPRINT -->
-<link name="base_footprint"/>
+<link name="base_link"/>
 <!-- Base Scan -->
 <link name="base_scan"/>
 <!-- chassis -->
-<link name="base_link" >
+<link name="base_body" >
   <inertial>
     <origin xyz="${chassis_length/2 - wheel_radius} 0 0" rpy="0 0 0"/>
-    <mass value="${0.04}"/>
+    <mass value="${M}"/>
     <inertia ixx="${1/12*M*(chassis_length**2+chassis_thickness**2)}"  ixy="0"  ixz="0" iyy="${1/12*M*((wheel_base - wheel_width)**2+chassis_thickness**2)}" iyz="0" izz="${1/12*M*(chassis_length**2+(wheel_base - wheel_width)**2)}" />
   </inertial>
@@ -104,13 +104,12 @@
 <!-- joints -->
 <joint name="base" type="fixed">
-  <!-- <origin xyz="${-chassis_length/2 + chassis_length/2 - wheel_radius} 0 ${chassis_thickness/2 - wheel_axle_offset + wheel_radius}" rpy="0 0 0" /> -->
   <origin xyz="${-wheel_radius} 0 ${chassis_thickness/2 - wheel_axle_offset + wheel_radius}" rpy="0 0 0" />
-  <parent link="base_footprint"/>
-  <child link="base_link" />
+  <parent link="base_link"/>
+  <child link="base_body" />
 </joint>
 <joint name="base_lidar" type="fixed">
   <origin xyz="0 0 ${chassis_thickness/2}" rpy="0 0 0" />
   <axis xyz="0 1 0"/>
-  <parent link="base_link" />
+  <parent link="base_body" />
   <child link="base_scan" />
 </joint>
@@ -118,5 +117,5 @@
   <origin xyz="0 ${wheel_base/2} ${-chassis_thickness/2 + wheel_axle_offset}" rpy="0 0 0" />
   <axis xyz="0 1 0"/>
-  <parent link="base_link" />
+  <parent link="base_body" />
   <child link="left_wheel" />
 </joint>
@@ -124,10 +123,10 @@
   <origin xyz="0 ${-wheel_base/2} ${-chassis_thickness/2 + wheel_axle_offset}" rpy="0 0 0" />
   <axis xyz="0 1 0"/>
-  <parent link="base_link" />
+  <parent link="base_body" />
   <child link="right_wheel" />
 </joint>
 <joint name="caster_joint" type="fixed">
   <origin xyz="${chassis_length - wheel_radius - caster_radius} 0 ${-chassis_thickness/2 - caster_radius}" rpy="0 0 0" />
-  <parent link="base_link" />
+  <parent link="base_body" />
   <child link="caster" />
 </joint>

Commit message: raised base_scan up 0.5 cm

File: nuturtle_description/urdf/diff_drive.urdf.xacro (robot description, xacro)
@@ -109,5 +109,5 @@
 </joint>
 <joint name="base_lidar" type="fixed">
-  <origin xyz="0 0 ${chassis_thickness/2}" rpy="0 0 0" />
+  <origin xyz="0 0 ${chassis_thickness/2 + 0.005}" rpy="0 0 0" />
   <axis xyz="0 1 0"/>
   <parent link="base_body" />
