Commit message: plugin done

File: nuturtle_gazebo/urdf/diff_drive.gazebo.xacro (robot description, xacro)
@@ -2,4 +2,28 @@
 <robot name="diff_drive" xmlns:xacro="http://www.ros.org/wiki/xacro">
 <xacro:include filename="$(find nuturtle_description)/urdf/diff_drive.urdf.xacro"/>
+<xacro:property name="diff_params" value="${load_yaml('$(find nuturtle_description)/config/diff_params.yaml')}" />
+<xacro:property name="odometer_params" value="${load_yaml('$(find rigid2d)/config/odometer_params.yaml')}" />
+<xacro:property name="left_joint_name" value="${odometer_params['left_wheel_joint']}" />
+<xacro:property name="right_joint_name" value="${odometer_params['right_wheel_joint']}" />
+<xacro:property name="Hz" value="${200}" />
+<xacro:property name="wheel_cmd_topic" value="nuturtlebot/WheelCommands" />
+<xacro:property name="sensor_topic" value="nuturtlebot/SensorData" />
+<xacro:property name="encoder_ticks_per_rev" value="${diff_params['encoder_ticks_per_rev']}" />
+<xacro:property name="max_motor_rot_vel" value="${diff_params['max_rot_motor']}" />
+<xacro:property name="max_motor_power" value="${diff_params['max_motor_power']}" />
+<xacro:property name="max_motor_torque" value="${diff_params['max_motor_torque']}" />
+<gazebo>
+  <plugin name="turtle_drive_plugin" filename="libnuturtle_gazebo_plugin.so">
+    <left_wheel_joint>${left_joint_name}</left_wheel_joint>
+    <right_wheel_joint>${right_joint_name}</right_wheel_joint>
+    <sensor_frequency>${Hz}</sensor_frequency>
+    <wheel_cmd_topic>${wheel_cmd_topic}</wheel_cmd_topic>
+    <sensor_topic>${sensor_topic}</sensor_topic>
+    <encoder_ticks_per_rev>${encoder_ticks_per_rev}</encoder_ticks_per_rev>
+    <max_motor_rot_vel>${max_motor_rot_vel}</max_motor_rot_vel>
+    <max_motor_power>${max_motor_power}</max_motor_power>
+    <max_motor_torque>${max_motor_torque}</max_motor_torque>
+  </plugin>
+</gazebo>
 <gazebo reference="base_link">
   <material>Gazebo/TurquoiseGlowOutline</material>

Commit message: update base_footprint

File: nuturtle_gazebo/urdf/diff_drive.gazebo.xacro (robot description, xacro)
@@ -7,6 +7,6 @@
 <xacro:property name="right_joint_name" value="${odometer_params['right_wheel_joint']}" />
 <xacro:property name="Hz" value="${200}" />
-<xacro:property name="wheel_cmd_topic" value="nuturtlebot/WheelCommands" />
-<xacro:property name="sensor_topic" value="nuturtlebot/SensorData" />
+<xacro:property name="wheel_cmd_topic" value="wheel_cmd" />
+<xacro:property name="sensor_topic" value="sensor_data" />
 <xacro:property name="encoder_ticks_per_rev" value="${diff_params['encoder_ticks_per_rev']}" />
 <xacro:property name="max_motor_rot_vel" value="${diff_params['max_rot_motor']}" />
@@ -26,39 +26,29 @@
   </plugin>
 </gazebo>
-<gazebo reference="base_link">
+<gazebo reference="base_body">
   <material>Gazebo/TurquoiseGlowOutline</material>
 </gazebo>
 <gazebo reference="left_wheel">
-  <!--
-  <dampingFactor>0.1</dampingFactor> -->
   <mu1>100</mu1>
   <mu2>100</mu2>
   <kp>500000.0</kp>
   <kd>10.0</kd>
-  <minDepth>0.001</minDepth>
   <maxVel>0.1</maxVel>
-  <fdir1>1 0 0</fdir1>
   <material>Gazebo/Red</material>
 </gazebo>
 <gazebo reference="right_wheel">
-  <!--
-  <dampingFactor>0.1</dampingFactor> -->
   <mu1>100</mu1>
   <mu2>100</mu2>
   <kp>500000.0</kp>
   <kd>10.0</kd>
-  <minDepth>0.001</minDepth>
   <maxVel>0.1</maxVel>
-  <fdir1>1 0 0</fdir1>
   <material>Gazebo/Red</material>
 </gazebo>
 <gazebo reference="caster">
-  <mu1>100</mu1>
-  <mu2>100</mu2>
+  <mu1>0.1</mu1>
+  <mu2>0.1</mu2>
   <kp>500000.0</kp>
   <kd>10.0</kd>
-  <minDepth>0.001</minDepth>
   <maxVel>0.1</maxVel>
-  <material>Gazebo/Red</material>
   <material>Gazebo/Black</material>
 </gazebo>

Commit message: lidar model added

File: nuturtle_gazebo/urdf/diff_drive.gazebo.xacro (robot description, xacro)
@@ -53,3 +53,35 @@
   <material>Gazebo/Black</material>
 </gazebo>
+<gazebo reference="base_scan">
+  <material>Gazebo/FlatBlack</material>
+  <sensor type="ray" name="lds_lfcd_sensor">
+    <pose>0 0 0 0 0 0</pose>
+    <visualize>true</visualize>
+    <update_rate>5</update_rate>
+    <ray>
+      <scan>
+        <horizontal>
+          <samples>360</samples>
+          <resolution>1</resolution>
+          <min_angle>0.0</min_angle>
+          <max_angle>6.28319</max_angle>
+        </horizontal>
+      </scan>
+      <range>
+        <min>0.120</min>
+        <max>3.5</max>
+        <resolution>0.015</resolution>
+      </range>
+      <noise>
+        <type>gaussian</type>
+        <mean>0.0</mean>
+        <stddev>0.01</stddev>
+      </noise>
+    </ray>
+    <plugin name="gazebo_ros_lds_lfcd_controller" filename="libgazebo_ros_laser.so">
+      <topicName>scan</topicName>
+      <frameName>base_scan</frameName>
+    </plugin>
+  </sensor>
+</gazebo>
 </robot>
